File: Hardware/SL869-GL868-Cx.brd (EAGLE design)
At the start: 133 parts, among them IC1 STM32F10XCXT6, Q1 IRLML6402, Q2 BC847/BSS138, Q5 IRF7353D2, U13 LP3985IM5-3.3, U14 GL865/8-DUAL, U15 SL868/9, U2 SIMHOLDER-MFF2, U4 SIMHOLDER-6393699, U5 MMA7455L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

Commit message: Cosmetic changes
Routing:
- net GND: vias 288 -> 289
Changed lines of the file:
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@@
 <setting verticaltext="up"/>
 </settings>
-<grid distance="0.2" unitdist="mm" unit="mm" style="lines" multiple="1" display="yes" altdistance="0.025" altunitdist="inch" altunit="inch"/>
+<grid distance="0.1" unitdist="mm" unit="mm" style="lines" multiple="1" display="yes" altdistance="0.025" altunitdist="inch" altunit="inch"/>
 <layers>
 <layer number="1" name="Top" color="4" fill="1" visible="yes" active="yes"/>
@@
 <via x="23" y="17" extent="1-16" drill="0.4"/>
 <via x="26.8" y="17" extent="1-16" drill="0.4"/>
-<via x="29.2" y="13.2" extent="1-16" drill="0.4"/>
+<via x="29.3" y="13.7" extent="1-16" drill="0.4"/>
 <contactref element="R5" pad="2"/>
 <contactref element="SV1" pad="2"/>
@@
 <via x="62.2" y="37.8" extent="1-16" drill="0.4"/>
 <via x="58.8" y="32.8" extent="1-16" drill="0.4"/>
-<via x="32" y="14.7" extent="1-16" drill="0.4"/>
+<via x="32.2" y="14.7" extent="1-16" drill="0.4"/>
 <via x="44.4" y="13.6" extent="1-16" drill="0.4"/>
-<via x="34.7" y="14" extent="1-16" drill="0.4"/>
+<via x="34.8" y="14.1" extent="1-16" drill="0.4"/>
 <via x="34.2" y="17.2" extent="1-16" drill="0.4"/>
 <contactref element="IC1" pad="28"/>
@@
 <via x="50.6" y="41" extent="1-16" drill="0.4"/>
 <via x="53" y="41" extent="1-16" drill="0.4"/>
+<via x="29.3" y="15.7" extent="1-16" drill="0.4"/>
 <wire x1="73.9" y1="13" x2="74" y2="13" width="0" layer="19" extent="1-16"/>
 </signal>
@@
 <contactref element="IC1" pad="9"/>
 <contactref element="IC1" pad="9"/>
-<wire x1="30.95" y1="12.95" x2="31.65" y2="12.95" width="0.25" layer="1"/>
-<wire x1="31.65" y1="12.95" x2="32" y2="13" width="0.25" layer="1"/>
-<via x="32" y="13" extent="1-16" drill="0.4"/>
-<wire x1="32" y1="13" x2="31.2" y2="13" width="0.25" layer="16"/>
+<wire x1="30.95" y1="12.95" x2="32.05" y2="12.95" width="0.25" layer="1"/>
+<wire x1="32.05" y1="12.95" x2="32.1" y2="13" width="0.25" layer="1"/>
+<via x="32.1" y="13" extent="1-16" drill="0.4"/>
+<wire x1="32.1" y1="13" x2="31.2" y2="13" width="0.25" layer="16"/>
 <wire x1="31.2" y1="13" x2="28" y2="9.8" width="0.25" layer="16"/>
 <wire x1="28" y1="9.8" x2="27.8" y2="9.8" width="0.25" layer="16"/>
@@
 <contactref element="C42" pad="1"/>
 <contactref element="IC1" pad="7"/>
-<wire x1="30.95" y1="13.95" x2="32.15" y2="13.95" width="0.2" layer="1"/>
-<wire x1="33.8" y1="12.3" x2="33.8" y2="11.6" width="0.2" layer="1"/>
-<via x="33.8" y="11.6" extent="1-16" drill="0.4"/>
+<wire x1="30.95" y1="13.95" x2="32.55" y2="13.95" width="0.2" layer="1"/>
+<wire x1="33.8" y1="12.7" x2="33.8" y2="11.5" width="0.2" layer="1"/>
+<via x="33.8" y="11.5" extent="1-16" drill="0.4"/>
 <contactref element="JP3" pad="4"/>
 <wire x1="33.02" y1="1.4" x2="33.02" y2="1.58" width="0.2" layer="16"/>
@@
 <via x="30" y="8.4" extent="1-16" drill="0.4"/>
 <wire x1="30" y1="8.4" x2="30.4" y2="8.4" width="0.2" layer="16"/>
-<wire x1="30.4" y1="8.4" x2="33.6" y2="11.6" width="0.2" layer="16"/>
-<wire x1="33.6" y1="11.6" x2="33.8" y2="11.6" width="0.2" layer="16"/>
+<wire x1="30.4" y1="8.4" x2="33.5" y2="11.5" width="0.2" layer="16"/>
+<wire x1="33.5" y1="11.5" x2="33.8" y2="11.5" width="0.2" layer="16"/>
 <wire x1="27.6" y1="8.35" x2="27.6" y2="8.4" width="0.2" layer="1"/>
 <wire x1="27.6" y1="8.4" x2="29.15" y2="8.4" width="0.2" layer="1"/>
@@
 <wire x1="29.2" y1="8.35" x2="29.2" y2="8.4" width="0.2" layer="1"/>
 <wire x1="29.2" y1="8.4" x2="30" y2="8.4" width="0.2" layer="1"/>
-<wire x1="33.8" y1="12.3" x2="32.15" y2="13.95" width="0.2" layer="1"/>
+<wire x1="33.8" y1="12.7" x2="32.55" y2="13.95" width="0.2" layer="1"/>
 </signal>
 <signal name="PB0.RELAY-ON">
@@
 <via x="36.8" y="13.4" extent="1-16" drill="0.4"/>
 <wire x1="36.8" y1="13.4" x2="36.2" y2="12.8" width="0.2" layer="16"/>
-<wire x1="36.2" y1="12.8" x2="33.4" y2="12.8" width="0.2" layer="16"/>
-<wire x1="33.4" y1="12.8" x2="32" y2="11.4" width="0.2" layer="16"/>
-<wire x1="32" y1="11.4" x2="31.2" y2="11.4" width="0.2" layer="16"/>
+<wire x1="36.2" y1="12.8" x2="33.5" y2="12.8" width="0.2" layer="16"/>
+<wire x1="33.5" y1="12.8" x2="32.1" y2="11.4" width="0.2" layer="16"/>
+<wire x1="32.1" y1="11.4" x2="31.2" y2="11.4" width="0.2" layer="16"/>
 <wire x1="31.2" y1="11.4" x2="28" y2="8.2" width="0.2" layer="16"/>
 <contactref element="RELAY" pad="P$1"/>
@@
 <via x="29.8" y="23.6" extent="1-16" drill="0.4"/>
 <contactref element="IC1" pad="18"/>
-<wire x1="34.95" y1="9.95" x2="34.95" y2="12.65" width="0.2" layer="1"/>
-<wire x1="34.95" y1="12.65" x2="33" y2="14.6" width="0.2" layer="1"/>
-<wire x1="33" y1="14.6" x2="33" y2="16.4" width="0.2" layer="1"/>
+<wire x1="34.95" y1="9.95" x2="34.95" y2="12.85" width="0.2" layer="1"/>
+<wire x1="34.95" y1="12.85" x2="33" y2="14.8" width="0.2" layer="1"/>
+<wire x1="33" y1="14.8" x2="33" y2="16.4" width="0.2" layer="1"/>
 <wire x1="33" y1="16.4" x2="32.2" y2="17.2" width="0.2" layer="1"/>
 <via x="32.2" y="17.2" extent="1-16" drill="0.4"/>
@@
 </signal>
 </signals>
-<errors>
-</errors>
 </board>
 </drawing>
