File: Hardware/SL869-GL868-Rx.brd (EAGLE design)
At the start: 82 x 41.4 mm, 196 parts, among them Q1 IRLML6402, Q10 8MHz, Q2 BC847/BSS138, Q5 IRF7353D2, Q6 IRLML6401, Q7 IRLML6401, SW1 SWT7, U1 74LVC1G02GV, U10 MAX1555, U11 STM32F103RBT6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

Commit message: Fix schematic/layout
Parts:
- D4: device X893:SOT-23@1 -> X893:SOT-23
Connections:
- removed net RXD1: U14.44
- removed net TXD1: U14.45
Routing:
- net N$2: track 0.80 -> 0.00 mm
Changed lines of the file:
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@@
 <?xml version="1.0" encoding="utf-8"?>
 <!DOCTYPE eagle SYSTEM "eagle.dtd">
-<eagle version="6.4">
+<eagle version="6.5.0">
 <drawing>
 <settings>
@@
 <element name="R20" library="X893" package="0603" value="22K" x="32.4" y="31.6" rot="R270"/>
 <element name="R21" library="X893" package="0603" value="22K" x="34" y="31.6" rot="R90"/>
-<element name="D4" library="X893" package="SOT-23@1" value="BAV99" x="14.8" y="14.4" rot="R270"/>
+<element name="D4" library="X893" package="SOT-23" value="BAV99" x="14.8" y="14.4" rot="R270"/>
 <element name="C13" library="X893" package="0603" value="0.1u" x="17.4" y="16.8"/>
 <element name="R26" library="X893" package="0603" value="100K" x="14.6" y="16.8"/>
@@
 <wire x1="27.6" y1="7.4" x2="26.6" y2="7.4" width="0.2" layer="1"/>
 </signal>
-<signal name="RXD1">
-<contactref element="U14" pad="44"/>
-</signal>
-<signal name="TXD1">
-<contactref element="U14" pad="45"/>
-</signal>
-<signal name="N$2">
-<wire x1="55.2" y1="20.8" x2="55.2" y2="20" width="0.2" layer="16"/>
-</signal>
 <signal name="N$20">
