File: Hardware/SL869-GL868-Cx.sch (EAGLE design)
At the start: 132 parts, among them IC1 STM32F10XCXT6, Q1 IRLML6402, Q2 BC847/BSS138, Q5 IRF7353D2, U13 LP3985IM5-3.3, U14 GL865/8-DUAL, U15 SL868/9, U2 SIMHOLDER-MFF2, U4 SIMHOLDER-6393699, U5 MMA7455L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

Commit message: Fix error with LED on PB3/PB4 with Cx version
Parts:
- DTR-DSR: value (none) -> DTR-DSR
- GPS-RXD: value (none) -> GPS-RXD
- GPS-TXD: value (none) -> GPS-TXD
- GSM-RESET: value (none) -> GSM-RESET
- Q4: value (none) -> 8MHz
- RTS-CTS: value (none) -> RTS-CTS
Connections:
- removed net GSM-DCD: U14.C109/DCD/GPO_A
- removed net GSM-RI: U14.C125/RING/GPO_B
Other:
- moved on the sheet: C56, C57, DTR-DSR, J1, J2, JP4, Q4
